Commit message: Updated amr_ros2_control.xacro and other files

File: src/amr_description/urdf/amr_ros2_control.xacro (robot description, xacro)
@@ -1,29 +1,15 @@
 <?xml version="1.0"?>
 <robot xmlns:xacro="http://ros.org/wiki/xacro" name="amr_robot">
-  <!-- Define the missing macro properly -->
-  <xacro:macro name="amr_ros2_control" params="is_sim is_ignition">
-    <ros2_control name="amr_robot_controller" type="system">
-      <!-- ros2_control Gazebo -->
-      <xacro:if value="${is_sim}">
-        <!-- ROS 2 Humble -->
-        <xacro:if value="${is_ignition}">
+  <ros2_control name="RobotSystem" type="system">
+       <xacro:if value="$(arg is_ignition)">
           <hardware>
             <plugin>ign_ros2_control/IgnitionSystem</plugin>
           </hardware>
         </xacro:if>
-        <!-- ROS 2 Iron or above -->
-        <xacro:unless value="${is_ignition}">
+        <xacro:unless value="$(arg is_ignition)">
           <hardware>
             <plugin>gz_ros2_control/GazeboSimSystem</plugin>
           </hardware>
         </xacro:unless>
-      </xacro:if>
-      <!-- ros2_control Real Robot -->
-      <xacro:unless value="${is_sim}">
-        <hardware>
-          <plugin>amr_bot_firmware/amr_botInterface</plugin>
-          <param name="port">/dev/ttyUSB0</param>
-        </hardware>
-      </xacro:unless>
       <!-- ros2_control Common Interfaces -->
       <joint name="wheel_right_joint">
@@ -44,4 +30,3 @@
       </joint>
     </ros2_control>
-  </xacro:macro>
 </robot>

Commit message: Updated AMR controller, description, and examples

File: src/amr_description/urdf/amr_ros2_control.xacro (robot description, xacro)
@@ -1,9 +1,9 @@
 <?xml version="1.0"?>
-<robot xmlns:xacro="http://ros.org/wiki/xacro">
+<robot name="amr_robot" xmlns:xacro="http://www.ros.org/wiki/xacro">
   <!-- Define the ros2_control configuration -->
-  <xacro:macro name="amr_ros2_control" params="is_sim is_ignition">
+    <xacro:macro name="amr_ros2_control" params="is_sim is_ignition">
     <ros2_control name="RobotSystem" type="gazebo_ros2_control">
       <!-- Use Ignition plugin if is_ignition=true -->
-      <xacro:if value="$(arg is_ignition)">
+      <xacro:if value="${is_ignition}">
         <hardware>
           <plugin>ign_ros2_control/IgnitionSystem</plugin>
@@ -11,5 +11,5 @@
       </xacro:if>
       <!-- Use Gazebo plugin if is_ignition=false -->
-      <xacro:unless value="$(arg is_ignition)">
+      <xacro:unless value="${is_ignition}">
         <hardware>
           <plugin>gazebo_ros2_control/GazeboSystem</plugin>
@@ -36,3 +36,4 @@
     </ros2_control>
   </xacro:macro>
+<xacro:amr_ros2_control is_sim="true" is_ignition="false"/>
 </robot>
