Commit message: Updated URDF and package.xml, removed unnecessary files

File: src/amr_description/urdf/amr.urdf.xacro (robot description, xacro)
@@ -1,18 +1,16 @@
 <?xml version="1.0"?>
-<robot name="amr_robot" xmlns:xacro="http://ros.org/wiki/xacro">
-  <!-- Start GZ or Ignition depending on ROS 2 Version -->
+<robot xmlns:xacro="http://ros.org/wiki/xacro" name="amr_robot">
+  <!--  Define Arguments -->
   <xacro:arg name="is_ignition" default="true"/>
   <xacro:arg name="is_sim" default="true"/>
-  <!-- Include Gazebo Parameters -->
-  <xacro:include filename="$(find amr_description)/urdf/amr_gazebo.xacro" />
   <!-- Include the ros2_control file -->
   <xacro:include filename="$(find amr_description)/urdf/amr_ros2_control.xacro" />
-  <!-- Call the macro with appropriate arguments (Correct usage) -->
-  <xacro:amr_ros2_control is_sim="$(arg is_sim)" is_ignition="$(arg is_ignition)"/>
-<gazebo>
-  <plugin name="gazebo_ros2_control" filename="libgazebo_ros2_control.so">
-    <robot_param>robot_description</robot_param>
-  </plugin>
-</gazebo>
+  <!-- Call the Macro After Including -->
+  <xacro:amr_ros2_control is_sim="${is_sim}" is_ignition="${is_ignition}"/>
+  <gazebo>
+    <plugin name="gazebo_ros2_control" filename="libgazebo_ros2_control.so">
+      <robot_param>robot_description</robot_param>
+    </plugin>
+  </gazebo>
 <link name="base_footprint"/>
 <link name="base_link">

File: src/amr_description/urdf/amr_ros2_control.xacro (robot description, xacro)
@@ -1,15 +1,17 @@
 <?xml version="1.0"?>
 <robot xmlns:xacro="http://ros.org/wiki/xacro" name="amr_robot">
-  <ros2_control name="RobotSystem" type="system">
-       <xacro:if value="$(arg is_ignition)">
-          <hardware>
-            <plugin>ign_ros2_control/IgnitionSystem</plugin>
-          </hardware>
-        </xacro:if>
-        <xacro:unless value="$(arg is_ignition)">
-          <hardware>
-            <plugin>gz_ros2_control/GazeboSimSystem</plugin>
-          </hardware>
-        </xacro:unless>
+  <xacro:macro name="amr_ros2_control" params="is_sim is_ignition">
+    <ros2_control name="RobotSystem" type="system">
+      <!-- Corrected condition handling -->
+      <xacro:if value="${is_ignition}">
+        <hardware>
+          <plugin>ign_ros2_control/IgnitionSystem</plugin>
+        </hardware>
+      </xacro:if>
+      <xacro:unless value="${is_ignition}">
+        <hardware>
+          <plugin>gz_ros2_control/GazeboSimSystem</plugin>
+        </hardware>
+      </xacro:unless>
       <!-- ros2_control Common Interfaces -->
       <joint name="wheel_right_joint">
@@ -30,3 +32,4 @@
       </joint>
     </ros2_control>
+  </xacro:macro>
 </robot>

Commit message: Updated AMR controller and description, cleaned logs

File: src/amr_description/urdf/amr.urdf.xacro (robot description, xacro)
@@ -1,17 +1,13 @@
 <?xml version="1.0"?>
-<robot xmlns:xacro="http://ros.org/wiki/xacro" name="amr_robot">
-  <!--  Define Arguments -->
+<robot name="bumperbot" xmlns:xacro="http://ros.org/wiki/xacro">
+  <!-- Start GZ or Ignition depending on ROS 2 Version -->
   <xacro:arg name="is_ignition" default="true"/>
-  <xacro:arg name="is_sim" default="true"/>
-  <!-- Include the ros2_control file -->
+  <!-- Load Simulated or Real Hardware Interfaces -->
+  <xacro:arg name="is_sim" default="false"/>
+  <!-- Include Gazebo Parameters -->
+  <xacro:include filename="$(find amr_description)/urdf/amr_gazebo.xacro" />
+  <!-- Include ros2_control Plugins -->
   <xacro:include filename="$(find amr_description)/urdf/amr_ros2_control.xacro" />
-  <!-- Call the Macro After Including -->
-  <xacro:amr_ros2_control is_sim="${is_sim}" is_ignition="${is_ignition}"/>
-  <gazebo>
-    <plugin name="gazebo_ros2_control" filename="libgazebo_ros2_control.so">
-      <robot_param>robot_description</robot_param>
-    </plugin>
-  </gazebo>
-<link name="base_footprint"/>
+  <link name="base_footprint"/>
 <link name="base_link">
 <inertial>

File: src/amr_description/urdf/amr_ros2_control.xacro (robot description, xacro)
@@ -1,35 +1,36 @@
 <?xml version="1.0"?>
-<robot xmlns:xacro="http://ros.org/wiki/xacro" name="amr_robot">
+<robot xmlns:xacro="http://ros.org/wiki/xacro">
   <xacro:macro name="amr_ros2_control" params="is_sim is_ignition">
     <ros2_control name="RobotSystem" type="system">
-      <!-- Corrected condition handling -->
-      <xacro:if value="${is_ignition}">
-        <hardware>
-          <plugin>ign_ros2_control/IgnitionSystem</plugin>
-        </hardware>
-      </xacro:if>
-      <xacro:unless value="${is_ignition}">
-        <hardware>
-          <plugin>gz_ros2_control/GazeboSimSystem</plugin>
-        </hardware>
-      </xacro:unless>
-      <!-- ros2_control Common Interfaces -->
-      <joint name="wheel_right_joint">
-        <command_interface name="velocity">
-          <param name="min">-1</param>
-          <param name="max">1</param>
-        </command_interface>
-        <state_interface name="position" />
-        <state_interface name="velocity" />
-      </joint>
-      <joint name="wheel_left_joint">
-        <command_interface name="velocity">
-          <param name="min">-1</param>
-          <param name="max">1</param>
-        </command_interface>
-        <state_interface name="position" />
-        <state_interface name="velocity" />
-      </joint>
-    </ros2_control>
-  </xacro:macro>
+    <!-- Use Ignition plugin if is_ignition=true -->
+    <xacro:if value="${is_ignition}">
+      <hardware>
+        <plugin>ign_ros2_control/SystemInterface</plugin>
+      </hardware>
+    </xacro:if>
+    <!-- Use Gazebo plugin if is_ignition=false -->
+    <xacro:unless value="${is_ignition}">
+      <hardware>
+        <plugin>gazebo_ros2_control/GazeboSystem</plugin>
+      </hardware>
+    </xacro:unless>
+    <!-- ros2_control Common Interfaces -->
+    <joint name="wheel_right_joint">
+      <command_interface name="velocity">
+        <param name="min">-1</param>
+        <param name="max">1</param>
+      </command_interface>
+      <state_interface name="position" />
+      <state_interface name="velocity" />
+    </joint>
+    <joint name="wheel_left_joint">
+      <command_interface name="velocity">
+        <param name="min">-1</param>
+        <param name="max">1</param>
+      </command_interface>
+      <state_interface name="position" />
+      <state_interface name="velocity" />
+    </joint>
+  </ros2_control>
+</xacro:macro>
 </robot>

Commit message: Updated URDF, launch files, and controller configuration

File: src/amr_description/urdf/amr.urdf.xacro (robot description, xacro)
@@ -1,4 +1,4 @@
 <?xml version="1.0"?>
-<robot name="bumperbot" xmlns:xacro="http://ros.org/wiki/xacro">
+<robot name="amr_bot" xmlns:xacro="http://ros.org/wiki/xacro">
   <!-- Start GZ or Ignition depending on ROS 2 Version -->
   <xacro:arg name="is_ignition" default="true"/>
@@ -9,4 +9,6 @@
   <!-- Include ros2_control Plugins -->
   <xacro:include filename="$(find amr_description)/urdf/amr_ros2_control.xacro" />
+  <!-- Call the ros2_control macro -->
+  <xacro:amr_ros2_control is_sim="$( arg is_sim)" is_ignition="$(arg is_ignition)"/>
   <link name="base_footprint"/>
 <link name="base_link">

File: src/amr_description/urdf/amr_gazebo.xacro (robot description, xacro)
@@ -55,11 +55,13 @@
   <!-- ROS 2 Control -->
   <gazebo>
+    <!-- Ignition plugin for ROS2 Control -->
     <xacro:if value="$(arg is_ignition)">
-      <plugin filename="ign_ros2_control-system" name="ign_ros2_control::IgnitionROS2ControlPlugin">
+        <plugin filename="libign_ros2_control-system.so" name="ign_ros2_control::IgnitionROS2ControlPlugin">
         <parameters>$(find amr_controller)/config/amr_controllers.yaml</parameters>
       </plugin>
     </xacro:if>
+    <!-- Gazebo plugin for ROS2 Control -->
     <xacro:unless value="$(arg is_ignition)">
-      <plugin filename="gz_ros2_control-system" name="gz_ros2_control::GazeboSimROS2ControlPlugin">
+        <plugin filename="libgz_ros2_control-system.so" name="gz_ros2_control::GazeboSimROS2ControlPlugin">
         <parameters>$(find amr_controller)/config/amr_controllers.yaml</parameters>
       </plugin>

File: src/amr_description/urdf/amr_ros2_control.xacro (robot description, xacro)
@@ -1,36 +1,38 @@
 <?xml version="1.0"?>
 <robot xmlns:xacro="http://ros.org/wiki/xacro">
+  <!-- Define the ros2_control configuration -->
   <xacro:macro name="amr_ros2_control" params="is_sim is_ignition">
-    <ros2_control name="RobotSystem" type="system">
-    <!-- Use Ignition plugin if is_ignition=true -->
-    <xacro:if value="${is_ignition}">
-      <hardware>
-        <plugin>ign_ros2_control/SystemInterface</plugin>
-      </hardware>
-    </xacro:if>
-    <!-- Use Gazebo plugin if is_ignition=false -->
-    <xacro:unless value="${is_ignition}">
-      <hardware>
-        <plugin>gazebo_ros2_control/GazeboSystem</plugin>
-      </hardware>
-    </xacro:unless>
-    <!-- ros2_control Common Interfaces -->
-    <joint name="wheel_right_joint">
-      <command_interface name="velocity">
-        <param name="min">-1</param>
-        <param name="max">1</param>
-      </command_interface>
-      <state_interface name="position" />
-      <state_interface name="velocity" />
-    </joint>
-    <joint name="wheel_left_joint">
-      <command_interface name="velocity">
-        <param name="min">-1</param>
-        <param name="max">1</param>
-      </command_interface>
-      <state_interface name="position" />
-      <state_interface name="velocity" />
-    </joint>
-  </ros2_control>
-</xacro:macro>
+    <ros2_control name="RobotSystem" type="gazebo_ros2_control">
+      <!-- Use Ignition plugin if is_ignition=true -->
+      <xacro:if value="$(arg is_ignition)">
+        <hardware>
+          <plugin>ign_ros2_control/IgnitionSystem</plugin>
+        </hardware>
+      </xacro:if>
+      <!-- Use Gazebo plugin if is_ignition=false -->
+      <xacro:unless value="$(arg is_ignition)">
+        <hardware>
+          <plugin>gazebo_ros2_control/GazeboSystem</plugin>
+        </hardware>
+      </xacro:unless>
+      <joint name="wheel_right_joint">
+        <command_interface name="velocity">
+          <param name="min">-1</param>
+          <param name="max">1</param>
+        </command_interface>
+        <state_interface name="position" />
+        <state_interface name="velocity" />
+        <state_interface name="effort" />
+      </joint>
+      <joint name="wheel_left_joint">
+        <command_interface name="velocity">
+          <param name="min">-1</param>
+          <param name="max">1</param>
+        </command_interface>
+        <state_interface name="position" />
+        <state_interface name="velocity" />
+        <state_interface name="effort" />
+      </joint>
+    </ros2_control>
+  </xacro:macro>
 </robot>

Commit message: Updated controller, URDF, and parameter scripts

File: src/amr_description/urdf/amr.urdf.xacro (robot description, xacro)
@@ -13,219 +13,219 @@
   <link name="base_footprint"/>
 <link name="base_link">
-<inertial>
+  <inertial>
 <!-- Slightly increase the mass for better stability -->
-<origin xyz="0 0 0.1" rpy="0.0 0.0 0.0"/>
-<mass value="1.2"/>
+    <origin xyz="0 0 0.1" rpy="0.0 0.0 0.0"/>
+    <mass value="1.2"/>
 <!-- Increased from 0.82573504 -->
-<inertia ixx="0.03" ixy="-0.0001" ixz="0.0003" iyy="0.03" iyz="-0.00005" izz="0.025"/>
-</inertial>
-<visual>
-<geometry>
-<box size="1.195 0.925 0.385"/>
+    <inertia ixx="0.03" ixy="-0.0001" ixz="0.0003" iyy="0.03" iyz="-0.00005" izz="0.025"/>
+  </inertial>
+  <visual>
+    <geometry>
+      <box size="1.195 0.925 0.385"/>
 <!-- Slightly increased height for center of gravity -->
-</geometry>
-<origin xyz="0 0 0.1" rpy="0 0 0"/>
-<material name="Green">
-  <color rgba="0 1 0 1"/> <!-- Green color (R,G,B,A) -->
-</material>
-</visual>
-<collision>
-<geometry>
-<box size="1.195 0.925 0.385"/>
-</geometry>
-<origin xyz="0 0 0.1" rpy="0 0 0"/>
-</collision>
+    </geometry>
+    <origin xyz="0 0 0.1" rpy="0 0 0"/>
+  <material name="Green">
+    <color rgba="0 1 0 1"/> <!-- Green color (R,G,B,A) -->
+  </material>
+  </visual>
+  <collision>
+    <geometry>
+      <box size="1.195 0.925 0.385"/>
+    </geometry>
+    <origin xyz="0 0 0.1" rpy="0 0 0"/>
+  </collision>
 </link>
 <link name="lidar">
-<inertial>
-<origin xyz="0 0 0" rpy="0 0 0"/>
-<mass value="0.6"/>
+  <inertial>
+    <origin xyz="0 0 0" rpy="0 0 0"/>
+    <mass value="0.6"/>
 <!-- Slightly increased mass for stability -->
-<inertia ixx="0.0006" ixy="0" ixz="0" iyy="0.0006" iyz="0" izz="0.0006"/>
-</inertial>
-<visual>
-<geometry>
-<cylinder radius="0.1" length="0.05"/>
-</geometry>
-<material name="red">
-  <color rgba="1 0 0 1"/>
-</material>
-<origin xyz="0 0 0.1" rpy="0 0 0"/>
-</visual>
-<collision>
-<geometry>
-<cylinder radius="0.1" length="0.05"/>
-</geometry>
-<origin xyz="0 0 0.1" rpy="0 0 0"/>
-</collision>
+    <inertia ixx="0.0006" ixy="0" ixz="0" iyy="0.0006" iyz="0" izz="0.0006"/>
+  </inertial>
+  <visual>
+  <geometry>
+    <cylinder radius="0.1" length="0.05"/>
+  </geometry>
+  <material name="red">
+    <color rgba="1 0 0 1"/>
+  </material>
+  <origin xyz="0 0 0.1" rpy="0 0 0"/>
+  </visual>
+  <collision>
+    <geometry>
+      <cylinder radius="0.1" length="0.05"/>
+    </geometry>
+    <origin xyz="0 0 0.1" rpy="0 0 0"/>
+  </collision>
 </link>
 <link name="wheel_left_link">
-<inertial>
-<origin xyz="0 0 0" rpy="0 0 0"/>
-<mass value="0.065"/>
-<!-- Increased mass for wheels to improve control -->
-<inertia ixx="0.00002" ixy="0" ixz="0" iyy="0.00004" iyz="0" izz="0.00002"/>
-</inertial>
-<visual>
-<geometry>
-<cylinder radius="0.09" length="0.06"/>
-<!-- Slightly larger wheel for better grip -->
-</geometry>
-<origin xyz="0 0 0" rpy="1.57 0 0"/>
-</visual>
-<collision>
-<geometry>
-<cylinder radius="0.08" length="0.05"/>
-</geometry>
-<origin xyz="0 0 0" rpy="1.57 0 0"/>
-</collision>
+  <inertial>
+    <origin xyz="0 0 0" rpy="0 0 0"/>
+    <mass value="0.065"/> <!-- Increased mass for wheels to improve control -->
+    <inertia ixx="0.00002" ixy="0" ixz="0" iyy="0.00004" iyz="0" izz="0.00002" />
+  </inertial>
+  <visual>
+    <geometry>
+      <cylinder radius="0.09" length="0.06"/> <!-- Slightly larger wheel for better grip -->
+    </geometry>
+    <origin xyz="0 0 0" rpy="1.57 0 0"/>
+  </visual>
+  <collision>
+    <geometry>
+      <cylinder radius="0.08" length="0.05"/>
+    </geometry>
+    <origin xyz="0 0 0" rpy="1.57 0 0"/>
+  </collision>
 </link>
 <link name="wheel_right_link">
-<inertial>
-<origin xyz="0 0 0" rpy="0 0 0"/>
-<mass value="0.065"/>
+  <inertial>
+    <origin xyz="0 0 0" rpy="0 0 0"/>
+    <mass value="0.065"/>
 <!-- Match mass for left and right wheels -->
-<inertia ixx="0.00002" ixy="0" ixz="0" iyy="0.00004" iyz="0" izz="0.00002"/>
-</inertial>
-<visual>
-<geometry>
-<cylinder radius="0.08" length="0.05"/>
-</geometry>
-<origin xyz="0 0 0" rpy="-1.57 0 0"/>
-</visual>
-<collision>
-<geometry>
-<cylinder radius="0.09" length="0.06"/>
-</geometry>
-<origin xyz="0 0 0" rpy="-1.57 0 0"/>
-</collision>
+    <inertia ixx="0.00002" ixy="0" ixz="0" iyy="0.00004" iyz="0" izz="0.00002"/>
+  </inertial>
+  <visual>
+    <geometry>
+      <cylinder radius="0.09" length="0.06"/>
+    </geometry>
+    <origin xyz="0 0 0" rpy="-1.57 0 0"/>
+  </visual>
+  <collision>
+    <geometry>
+      <cylinder radius="0.08" length="0.05"/>
+    </geometry>
+    <origin xyz="0 0 0" rpy="-1.57 0 0"/>
+  </collision>
 </link>
 <link name="caster_wheel_front">
-<inertial>
-<origin xyz="0 0 0" rpy="0 0 0"/>
-<mass value="0.00144379265037902"/>
-<inertia ixx="0.0000000000723075276010246" ixy="0" ixz="0" iyy="0.0000000000387137930859167" iyz="0" izz="0.000000000100967486676306"/>
-</inertial>
-<visual>
-<geometry>
-<cylinder radius="0.08" length="0.05"/>
-</geometry>
-<origin xyz="0 0 0" rpy="-1.57 0 0"/>
-</visual>
-<collision>
-<geometry>
-<sphere radius="0.08"/>
-</geometry>
-<origin xyz="0 0 0" rpy="0 0 0"/>
-</collision>
+  <inertial>
+    <origin xyz="0 0 0" rpy="0 0 0"/>
+    <mass value="0.00144379265037902"/>
+    <inertia ixx="0.0000000000723075276010246" ixy="0" ixz="0" iyy="0.0000000000387137930859167" iyz="0" izz="0.000000000100967486676306"/>
+  </inertial>
+  <visual>
+    <geometry>
+      <cylinder radius="0.08" length="0.05"/>
+    </geometry>
+    <origin xyz="0 0 0" rpy="-1.57 0 0"/>
+  </visual>
+  <collision>
+    <geometry>
+      <sphere radius="0.08"/>
+    </geometry>
+    <origin xyz="0 0 0" rpy="0 0 0"/>
+  </collision>
 </link>
 <link name="caster_wheel_rear">
-<inertial>
-<origin xyz="0 0 0" rpy="0 0 0"/>
-<mass value="0.00144379265037902"/>
-<inertia ixx="0.0000000000723075276010246" ixy="0" ixz="0" iyy="0.0000000000387137930859167" iyz="0" izz="0.000000000100967486676306"/>
-</inertial>
-<visual>
-<geometry>
-<cylinder radius="0.08" length="0.05"/>
-</geometry>
-<origin xyz="0 0 0" rpy="-1.57 0 0"/>
-</visual>
-<collision>
-<geometry>
-<sphere radius="0.08"/>
-</geometry>
-<origin xyz="0 0 0" rpy="0 0 0"/>
-</collision>
+  <inertial>
+    <origin xyz="0 0 0" rpy="0 0 0"/>
+    <mass value="0.00144379265037902"/>
+    <inertia ixx="0.0000000000723075276010246" ixy="0" ixz="0" iyy="0.0000000000387137930859167" iyz="0" izz="0.000000000100967486676306"/>
+  </inertial>
+  <visual>
+    <geometry>
+      <cylinder radius="0.08" length="0.05"/>
+    </geometry>
+    <origin xyz="0 0 0" rpy="-1.57 0 0"/>
+  </visual>
+  <collision>
+    <geometry>
+      <sphere radius="0.08"/>
+    </geometry>
+    <origin xyz="0 0 0" rpy="0 0 0"/>
+  </collision>
 </link>
 <link name="caster1_wheel_front">
-<inertial>
-<origin xyz="0 0 0" rpy="0 0 0"/>
-<mass value="0.00144379265037902"/>
-<inertia ixx="0.0000000000723075276010246" ixy="0" ixz="0" iyy="0.0000000000387137930859167" iyz="0" izz="0.000000000100967486676306"/>
-</inertial>
-<visual>
-<geometry>
-<cylinder radius="0.08" length="0.05"/>
-</geometry>
-<origin xyz="0 0 0" rpy="-1.57 0 0"/>
-</visual>
-<collision>
-<geometry>
-<sphere radius="0.05"/>
-</geometry>
-<origin xyz="0 0 0" rpy="0 0 0"/>
-</collision>
+  <inertial>
+    <origin xyz="0 0 0" rpy="0 0 0"/>
+    <mass value="0.00144379265037902"/>
+    <inertia ixx="0.0000000000723075276010246" ixy="0" ixz="0" iyy="0.0000000000387137930859167" iyz="0" izz="0.000000000100967486676306"/>
+  </inertial>
+  <visual>
+    <geometry>
+      <cylinder radius="0.08" length="0.05"/>
+    </geometry>
+    <origin xyz="0 0 0" rpy="-1.57 0 0"/>
+  </visual>
+  <collision>
+    <geometry>
+      <sphere radius="0.05"/>
+    </geometry>
+    <origin xyz="0 0 0" rpy="0 0 0"/>
+  </collision>
 </link>
 <link name="caster2_wheel_rear">
-<inertial>
-<origin xyz="0 0 0" rpy="0 0 0"/>
-<mass value="0.00144379265037902"/>
-<inertia ixx="0.0000000000723075276010246" ixy="0" ixz="0" iyy="0.0000000000387137930859167" iyz="0" izz="0.000000000100967486676306"/>
-</inertial>
-<visual>
-<geometry>
-<cylinder radius="0.08" length="0.05"/>
-</geometry>
-<origin xyz="0 0 0" rpy="-1.57 0 0"/>
-</visual>
-<collision>
-<geometry>
-<sphere radius="0.05"/>
-</geometry>
-<origin xyz="0 0 0" rpy="0 0 0"/>
-</collision>
+  <inertial>
+    <origin xyz="0 0 0" rpy="0 0 0"/>
+    <mass value="0.00144379265037902"/>
+    <inertia ixx="0.0000000000723075276010246" ixy="0" ixz="0" iyy="0.0000000000387137930859167" iyz="0" izz="0.000000000100967486676306"/>
+  </inertial>
+  <visual>
+    <geometry>
+      <cylinder radius="0.08" length="0.05"/>
+    </geometry>
+    <origin xyz="0 0 0" rpy="-1.57 0 0"/>
+  </visual>
+  <collision>
+    <geometry>
+      <sphere radius="0.05"/>
+    </geometry>
+    <origin xyz="0 0 0" rpy="0 0 0"/>
+  </collision>
 </link>
 <!-- Caster Wheels and other links remain unchanged -->
 <!-- Joints -->
 <joint name="base_joint" type="fixed">
-<parent link="base_footprint"/>
-<child link="base_link"/>
-<origin xyz="0 0 0.1" rpy="0 0 0"/>
+  <parent link="base_footprint"/>
+  <child link="base_link"/>
+  <origin xyz="0 0 0.1" rpy="0 0 0.033"/>
 </joint>
 <joint name="base_lidar_joint" type="fixed">
-<parent link="base_link"/>
-<child link="lidar"/>
-<origin xyz="0 0 0.15" rpy="0 0 0"/>
+  <parent link="base_link"/>
+  <child link="lidar"/>
+  <origin xyz="0 0 0.15" rpy="0 0 0"/>
 </joint>
 <!-- Fine-tuned joint parameters -->
 <joint name="wheel_right_joint" type="continuous">
-<parent link="base_link"/>
-<child link="wheel_right_link"/>
-<origin xyz="-0.05 0.34 -0.09" rpy="0 0 0"/>
+  <parent link="base_link"/>
+  <child link="wheel_right_link"/>
+  <origin xyz="-0.05 0.34 -0.09" rpy="0 0 0"/>
 <!-- Increased distance for better stability -->
-<axis xyz="0 1 0"/>
+  <axis xyz="0 1 0"/>
+  <dynamics damping="0.5" friction="1.0"/>
 </joint>
 <joint name="wheel_left_joint" type="continuous">
-<parent link="base_link"/>
-<child link="wheel_left_link"/>
-<origin xyz="-0.05 -0.34 -0.09" rpy="0 0 0"/>
+  <parent link="base_link"/>
+  <child link="wheel_left_link"/>
+  <origin xyz="-0.05 -0.34 -0.09" rpy="0 0 0"/>
 <!-- Symmetrical adjustment -->
-<axis xyz="0 1 0"/>
-</joint>
+  <axis xyz="0 1 0"/>
+  <dynamics damping="0.5" friction="1.0"/>
+  </joint>
 <!-- Rest of the caster wheel joints remain unchanged -->
 <joint name="front_caster_wheel_joint" type="fixed">
-<parent link="base_link"/>
-<child link="caster_wheel_front"/>
-<origin xyz="0.4 0.32 -0.09" rpy="0 0 0"/>
-<axis xyz="0 1 0"/>
+  <parent link="base_link"/>
+  <child link="caster_wheel_front"/>
+  <origin xyz="0.4 0.32 -0.09" rpy="0 0 0"/>
+  <axis xyz="0 1 0"/>
 </joint>
 <joint name="rear_caster_wheel_joint" type="fixed">
-<parent link="base_link"/>
-<child link="caster_wheel_rear"/>
-<origin xyz="0.4 -0.32 -0.09" rpy="0 0 0"/>
-<axis xyz="0 1 0"/>
+  <parent link="base_link"/>
+  <child link="caster_wheel_rear"/>
+  <origin xyz="0.4 -0.32 -0.09" rpy="0 0 0"/>
+  <axis xyz="0 1 0"/>
 </joint>
 <joint name="front_caster1_wheel_joint" type="fixed">
-<parent link="base_link"/>
-<child link="caster1_wheel_front"/>
-<origin xyz="-0.4 -0.32 -0.09" rpy="0 0 0"/>
-<axis xyz="0 1 0"/>
+  <parent link="base_link"/>
+  <child link="caster1_wheel_front"/>
+  <origin xyz="-0.4 -0.32 -0.09" rpy="0 0 0"/>
+  <axis xyz="0 1 0"/>
 </joint>
 <joint name="rear_caster2_wheel_joint" type="fixed">
-<parent link="base_link"/>
-<child link="caster2_wheel_rear"/>
-<origin xyz="-0.4 0.32 -0.09" rpy="0 0 0"/>
-<axis xyz="0 1 0"/>
+  <parent link="base_link"/>
+  <child link="caster2_wheel_rear"/>
+  <origin xyz="-0.4 0.32 -0.09" rpy="0 0 0"/>
+  <axis xyz="0 1 0"/>
 </joint>
 </robot>

File: src/amr_description/urdf/amr_gazebo.xacro (robot description, xacro)
@@ -3,6 +3,6 @@
   <!-- Middle Drive Wheels -->
   <gazebo reference="wheel_left_link">
-    <mu1>1000000000000000.0</mu1>
-    <mu2>1000000000000000.0</mu2>
+    <mu1>0.8</mu1>
+    <mu2>0.8</mu2>
     <kp>1000000000000.0</kp>
     <kd>10.0</kd>
@@ -12,6 +12,6 @@
   </gazebo>
   <gazebo reference="wheel_right_link">
-    <mu1>1000000000000000.0</mu1>
-    <mu2>1000000000000000.0</mu2>
+    <mu1>0.8</mu1>
+    <mu2>0.8</mu2>
     <kp>1000000000000.0</kp>
     <kd>10.0</kd>
