Commit message: Update controller configuration and URDF files

File: src/amr_description/urdf/amr.urdf.xacro (robot description, xacro)
@@ -16,12 +16,10 @@
 <!-- Slightly increase the mass for better stability -->
     <origin xyz="0 0 0.1" rpy="0.0 0.0 0.0"/>
-    <mass value="1.2"/>
-<!-- Increased from 0.82573504 -->
+    <mass value="1.2"/>   <!-- Increased from 0.82573504 -->
     <inertia ixx="0.03" ixy="-0.0001" ixz="0.0003" iyy="0.03" iyz="-0.00005" izz="0.025"/>
   </inertial>
   <visual>
     <geometry>
-      <box size="1.195 0.925 0.385"/>
-<!-- Slightly increased height for center of gravity -->
+      <box size="1.195 0.925 0.385"/>  <!-- Slightly increased height for center of gravity -->
     </geometry>
     <origin xyz="0 0 0.1" rpy="0 0 0"/>
@@ -40,6 +38,5 @@
   <inertial>
     <origin xyz="0 0 0" rpy="0 0 0"/>
-    <mass value="0.6"/>
-<!-- Slightly increased mass for stability -->
+    <mass value="0.6"/>  <!-- Slightly increased mass for stability -->
     <inertia ixx="0.0006" ixy="0" ixz="0" iyy="0.0006" iyz="0" izz="0.0006"/>
   </inertial>
@@ -63,10 +60,10 @@
   <inertial>
     <origin xyz="0 0 0" rpy="0 0 0"/>
-    <mass value="0.065"/> <!-- Increased mass for wheels to improve control -->
+    <mass value="0.065"/>  <!-- Increased mass for wheels to improve control -->
     <inertia ixx="0.00002" ixy="0" ixz="0" iyy="0.00004" iyz="0" izz="0.00002" />
   </inertial>
   <visual>
     <geometry>
-      <cylinder radius="0.09" length="0.06"/> <!-- Slightly larger wheel for better grip -->
+      <cylinder radius="0.08" length="0.06"/>  <!-- Slightly larger wheel for better grip -->
     </geometry>
     <origin xyz="0 0 0" rpy="1.57 0 0"/>
@@ -88,5 +85,5 @@
   <visual>
     <geometry>
-      <cylinder radius="0.09" length="0.06"/>
+      <cylinder radius="0.08" length="0.06"/>
     </geometry>
     <origin xyz="0 0 0" rpy="-1.57 0 0"/>
@@ -180,5 +177,5 @@
   <parent link="base_footprint"/>
   <child link="base_link"/>
-  <origin xyz="0 0 0.1" rpy="0 0 0.033"/>
+  <origin xyz="0 0 0.1" rpy="0 0 0"/>
 </joint>
 <joint name="base_lidar_joint" type="fixed">
@@ -191,16 +188,14 @@
   <parent link="base_link"/>
   <child link="wheel_right_link"/>
-  <origin xyz="-0.05 0.34 -0.09" rpy="0 0 0"/>
-<!-- Increased distance for better stability -->
-  <axis xyz="0 1 0"/>
-  <dynamics damping="0.5" friction="1.0"/>
+  <origin xyz="-0.05 0.34 -0.09" rpy="0 0 0"/>  <!-- Increased distance for better stability -->
+  <axis xyz="0 1 0"/>
+  <dynamics damping="0.1" friction="0.5"/>
 </joint>
 <joint name="wheel_left_joint" type="continuous">
   <parent link="base_link"/>
   <child link="wheel_left_link"/>
-  <origin xyz="-0.05 -0.34 -0.09" rpy="0 0 0"/>
-<!-- Symmetrical adjustment -->
-  <axis xyz="0 1 0"/>
-  <dynamics damping="0.5" friction="1.0"/>
+  <origin xyz="-0.05 -0.34 -0.09" rpy="0 0 0"/>  <!-- Symmetrical adjustment -->
+  <axis xyz="0 1 0"/>
+  <dynamics damping="0.1" friction="0.5"/>
   </joint>
 <!-- Rest of the caster wheel joints remain unchanged -->
@@ -229,3 +224,16 @@
   <axis xyz="0 1 0"/>
 </joint>
+<!-- Transmissions for ros2_control -->
+  <transmission name="left_wheel_transmission">
+    <type>transmission_interface/SimpleTransmission</type>
+    <joint name="wheel_left_joint">
+      <hardwareInterface>hardware_interface/VelocityJointInterface</hardwareInterface>
+    </joint>
+  </transmission>
+  <transmission name="right_wheel_transmission">
+    <type>transmission_interface/SimpleTransmission</type>
+    <joint name="wheel_right_joint">
+      <hardwareInterface>hardware_interface/VelocityJointInterface</hardwareInterface>
+    </joint>
+  </transmission>
 </robot>

File: src/amr_description/urdf/amr_gazebo.xacro (robot description, xacro)
@@ -1,4 +1,4 @@
 <?xml version="1.0"?>
-<robot name="amr_robot" xmlns:xacro="http://ros.org/wiki/xacro">
+<robot name="amr_bot" xmlns:xacro="http://ros.org/wiki/xacro">
   <!-- Middle Drive Wheels -->
   <gazebo reference="wheel_left_link">
@@ -53,4 +53,17 @@
     <maxVel>1.0</maxVel>
   </gazebo>
+<!-- Diff Drive Plugin (ADD THIS SECTION) -->
+  <gazebo>
+    <plugin filename="libgazebo_ros_diff_drive.so" name="diff_drive">
+      <ros>
+        <namespace>/amr_controller</namespace>
+        <remapping>cmd_vel:=cmd_vel</remapping>  <!-- Remove `/` in remapping -->
+      </ros>
+      <left_joint>left_wheel_joint</left_joint>
+      <right_joint>right_wheel_joint</right_joint>
+      <wheel_separation>0.322</wheel_separation>
+      <wheel_radius>0.08</wheel_radius>
+    </plugin>
+  </gazebo>
   <!-- ROS 2 Control -->
   <gazebo>

File: src/amr_description/urdf/amr_ros2_control.xacro (robot description, xacro)
@@ -1,4 +1,4 @@
 <?xml version="1.0"?>
-<robot name="amr_robot" xmlns:xacro="http://www.ros.org/wiki/xacro">
+<robot name="amr_bot" xmlns:xacro="http://www.ros.org/wiki/xacro">
   <!-- Define the ros2_control configuration -->
     <xacro:macro name="amr_ros2_control" params="is_sim is_ignition">

Commit message: Updated controller configurations, URDF files, and launch files

File: src/amr_description/urdf/amr.urdf.xacro (robot description, xacro)
@@ -48,5 +48,5 @@
     <color rgba="1 0 0 1"/>
   </material>
-  <origin xyz="0 0 0.1" rpy="0 0 0"/>
+  <origin xyz="0 0 0.15" rpy="0 0 0"/>
   </visual>
   <collision>
@@ -54,5 +54,5 @@
       <cylinder radius="0.1" length="0.05"/>
     </geometry>
-    <origin xyz="0 0 0.1" rpy="0 0 0"/>
+    <origin xyz="0 0 0.15" rpy="0 0 0"/>
   </collision>
 </link>

File: src/amr_description/urdf/amr_gazebo.xacro (robot description, xacro)
@@ -53,10 +53,10 @@
     <maxVel>1.0</maxVel>
   </gazebo>
-<!-- Diff Drive Plugin (ADD THIS SECTION) -->
+<!-- Diff Drive Plugin -->
   <gazebo>
     <plugin filename="libgazebo_ros_diff_drive.so" name="diff_drive">
       <ros>
         <namespace>/amr_controller</namespace>
-        <remapping>cmd_vel:=cmd_vel</remapping>  <!-- Remove `/` in remapping -->
+        <remapping>cmd_vel:=/amr_controller/cmd_vel</remapping>
       </ros>
       <left_joint>left_wheel_joint</left_joint>
@@ -64,4 +64,8 @@
       <wheel_separation>0.322</wheel_separation>
       <wheel_radius>0.08</wheel_radius>
+      <odom_frame>odom</odom_frame>
+      <robot_base_frame>base_link</robot_base_frame>
+      <update_rate>50</update_rate>
+      <max_wheel_torque>10.0</max_wheel_torque>
     </plugin>
   </gazebo>

Commit message: Integrated YDLIDAR driver, updated build logs, ignored log files

File: src/amr_description/urdf/amr.urdf.xacro (robot description, xacro)
@@ -224,4 +224,27 @@
   <axis xyz="0 1 0"/>
 </joint>
+<link name="imu_link">
+  <inertial>
+    <origin xyz="0 0 0" rpy="0 0 0"/>
+    <mass value="0.00144379265037902"/>
+    <inertia ixx="0.0000000000723075276010246" ixy="0" ixz="0" iyy="0.0000000000387137930859167" iyz="0" izz="0.000000000100967486676306"/>
+  </inertial>
+  <visual>
+   <origin xyz="0 0 0" rpy="0 0 0"/>
+   <geometry>
+   </geometry>
+  </visual>
+  <collision>
+    <origin xyz="0 0 0" rpy="0 0 0"/>
+  <geometry>
+  </geometry>
+  </collision>
+</link>
+<joint name="imu_joint" type="fixed">
+  <origin xyz="0 0 0" rpy="3.14 0 0"/>
+  <parent link="base_link"/>
+  <child link="imu_link"/>
+  <axis xyz="0 0 0"/>
+</joint>
 <!-- Transmissions for ros2_control -->
   <transmission name="left_wheel_transmission">

File: src/amr_description/urdf/amr_gazebo.xacro (robot description, xacro)
@@ -70,5 +70,5 @@
     </plugin>
   </gazebo>
-  <!-- ROS 2 Control -->
+   <!-- ROS 2 Control -->
   <gazebo>
     <!-- Ignition plugin for ROS2 Control -->
@@ -76,4 +76,6 @@
         <plugin filename="libign_ros2_control-system.so" name="ign_ros2_control::IgnitionROS2ControlPlugin">
         <parameters>$(find amr_controller)/config/amr_controllers.yaml</parameters>
+      </plugin>
+      <plugin filename="ignition-gazebo-imu-system" name="ignition::gazebo::systems::Imu">
       </plugin>
     </xacro:if>
@@ -83,5 +85,57 @@
         <parameters>$(find amr_controller)/config/amr_controllers.yaml</parameters>
       </plugin>
+      <plugin filename="gz-sim-imu-system" name="gz::sim::systems::Imu">
+      </plugin>
     </xacro:unless>
   </gazebo>
+  <gazebo reference="imu_link">
+    <sensor name="imu" type="imu">
+        <always_on>true</always_on>
+        <update_rate>100</update_rate>
+        <gz_frame_id>imu_link</gz_frame_id>
+        <topic>imu</topic>
+        <imu>
+          <angular_velocity>
+          <x>
+            <noise type="guassian">
+              <mean>0.0</mean>
+              <stddev>2e-4</stddev>
+            </noise>
+          </x>
+           <y>
+            <noise type="guassian">
+              <mean>0.0</mean>
+              <stddev>2e-4</stddev>
+            </noise>
+          </y>
+          <z>
+            <noise type="guassian">
+              <mean>0.0</mean>
+              <stddev>2e-4</stddev>
+            </noise>
+          </z>
+          </angular_velocity>
+          <linear_acceleration>
+            <x>
+              <noise type="guassian">
+                <mean>0.0</mean>
+                <stddev>1.7e-2</stddev>
+              </noise>
+            </x>
+            <y>
+              <noise type="guassian">
+                <mean>0.0</mean>
+                <stddev>1.7e-2</stddev>
+              </noise>
+            </y>
+            <z>
+              <noise type="guassian">
+                <mean>0.0</mean>
+                <stddev>1.7e-2</stddev>
+              </noise>
+            </z>
+          </linear_acceleration>
+          </imu>
+    </sensor>
+  </gazebo>
 </robot>

Commit message: Updated joystick teleop, added twist_mux configs, and updated URDF and LIDAR reader

File: src/amr_description/urdf/amr.urdf.xacro (robot description, xacro)
@@ -35,5 +35,5 @@
   </collision>
 </link>
-<link name="lidar">
+<link name="laser_link">
   <inertial>
     <origin xyz="0 0 0" rpy="0 0 0"/>
@@ -179,8 +179,8 @@
   <origin xyz="0 0 0.1" rpy="0 0 0"/>
 </joint>
-<joint name="base_lidar_joint" type="fixed">
-  <parent link="base_link"/>
-  <child link="lidar"/>
-  <origin xyz="0 0 0.15" rpy="0 0 0"/>
+<joint name="laser_joint" type="fixed">
+  <parent link="base_link"/>
+  <child link="laser_link"/>
+  <origin xyz="0.3 0 0.15" rpy="0 0 0"/>
 </joint>
 <!-- Fine-tuned joint parameters -->
@@ -238,4 +238,5 @@
     <origin xyz="0 0 0" rpy="0 0 0"/>
   <geometry>
+    <mesh filename="package://amr_description/meshes/imu_link.STL" />
   </geometry>
   </collision>

File: src/amr_description/urdf/amr_gazebo.xacro (robot description, xacro)
@@ -70,37 +70,4 @@
     </plugin>
   </gazebo>
-  <!-- Lidar Sensor Plugin -->
-  <gazebo reference="lidar">
-    <sensor name="lidar_sensor" type="ray">
-      <always_on>true</always_on>
-      <update_rate>10</update_rate>
-      <visualize>true</visualize>
-      <ray>
-        <scan>
-          <horizontal>
-            <samples>360</samples>
-            <resolution>1</resolution>
-            <min_angle>-3.14</min_angle>
-            <max_angle>3.14</max_angle>
-          </horizontal>
-        </scan>
-        <range>
-          <min>0.12</min>
-          <max>10.0</max>
-        </range>
-        <noise>
-          <type>gaussian</type>
-          <mean>0.0</mean>
-          <stddev>0.01</stddev>
-        </noise>
-      </ray>
-      <plugin name="lidar_plugin" filename="gz-sim-sensor-system">
-        <ros>
-          <remapping>~/scan:=/scan</remapping>
-        </ros>
-        <frameName>lidar</frameName>
-      </plugin>
-    </sensor>
-  </gazebo>
   <!-- ROS 2 Control -->
   <gazebo>
@@ -112,4 +79,7 @@
       <plugin filename="ignition-gazebo-imu-system" name="ignition::gazebo::systems::Imu">
       </plugin>
+      <plugin filename="ignition-gazebo-sensors-system" name="ignition::gazebo::systems::Sensors">
+        <render_engine>ogre2</render_engine>
+      </plugin>
     </xacro:if>
     <!-- Gazebo plugin for ROS2 Control -->
@@ -119,4 +89,7 @@
       </plugin>
       <plugin filename="gz-sim-imu-system" name="gz::sim::systems::Imu">
+      </plugin>
+      <plugin filename="gz-sim-sensors-system" name="gz::sim::systems::Sensors">
+        <render_engine>ogre2</render_engine>
       </plugin>
     </xacro:unless>
@@ -172,3 +145,39 @@
     </sensor>
   </gazebo>
+  <!-- Lidar Sensor Plugin -->
+  <gazebo reference="laser_link">
+    <sensor name="lidar" type="gpu_ray">
+      <always_on>true</always_on>
+      <update_rate>5</update_rate>
+      <topic>scan</topic>
+      <visualize>true</visualize>
+      <gz_frame_id>laser_link</gz_frame_id>
+      <ray>
+        <scan>
+          <horizontal>
+            <samples>360</samples>
+            <resolution>1.0</resolution>
+            <min_angle>0.0</min_angle>
+            <max_angle>6.28</max_angle>
+          </horizontal>
+        </scan>
+        <range>
+          <min>0.12</min>
+          <max>12.0</max>
+          <resolution>0.02</resolution>
+        </range>
+        <noise>
+          <type>gaussian</type>
+          <mean>0.0</mean>
+          <stddev>0.01</stddev>
+        </noise>
+      </ray>
+      <plugin name="lidar_plugin" filename="gz-sim-sensor-system">
+        <ros>
+          <remapping>~/scan:=/scan</remapping>
+        </ros>
+        <frameName>lidar</frameName>
+      </plugin>
+    </sensor>
+  </gazebo>
 </robot>
